File: board/sp3232e_TI-max232/SUNBoardSingleLayer.brd (EAGLE design)
At the start: 101.6 x 53.3 mm, 26 parts

Commit message: Fixed vias
Parts:
- added IOREF: (no value), pinhead:1X02
Changed lines of the file:
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@@
 <?xml version="1.0" encoding="utf-8"?>
 <!DOCTYPE eagle SYSTEM "eagle.dtd">
-<eagle version="6.6.0">
+<eagle version="6.5.0">
 <drawing>
 <settings>
@@
 <setting verticaltext="up"/>
 </settings>
-<grid distance="0.032258" unitdist="mm" unit="mm" style="lines" multiple="1" display="yes" altdistance="393.700787" altunitdist="mil" altunit="mil"/>
+<grid distance="1.27" unitdist="mm" unit="mm" style="lines" multiple="1" display="yes" altdistance="2.54" altunitdist="mil" altunit="mil"/>
 <layers>
 <layer number="1" name="Top" color="4" fill="1" visible="yes" active="yes"/>
@@
 <attribute name="VALUE" x="17.526" y="47.625" size="1.27" layer="27"/>
 </element>
+<element name="IOREF" library="pinhead" package="1X02" value="" x="29.21" y="2.54" locked="yes" smashed="yes">
+<attribute name="VALUE" x="26.67" y="-0.635" size="1.27" layer="27"/>
+</element>
 </elements>
